File: XmasTreeCard.brd (EAGLE design)
At the start: 153.7 x 92.9 mm, 51 parts, among them SW1 SWITCH_SPST6X6TACTILE

Commit message: Added CC BY-SA 4.0 License
Parts:
- added U$6: (no value), SparkFun-Aesthetics:OSHW-LOGO-M
Other:
- board text added: "CC BY-SA 4.0 http://github.com/mjholmes"
- board text added: "XmasCard v1.1"
- board text removed: "XmasCard v1"
Changed lines of the file:
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@@
 <layer number="20" name="Dimension" color="15" fill="1" visible="yes" active="yes"/>
 <layer number="21" name="tPlace" color="7" fill="1" visible="yes" active="yes"/>
-<layer number="22" name="bPlace" color="7" fill="1" visible="yes" active="yes"/>
+<layer number="22" name="bPlace" color="7" fill="1" visible="no" active="yes"/>
 <layer number="23" name="tOrigins" color="15" fill="1" visible="no" active="yes"/>
 <layer number="24" name="bOrigins" color="15" fill="1" visible="no" active="yes"/>
@@
 <rectangle x1="45.011846875" y1="35.8275" x2="45.208746875" y2="35.83346875" layer="21"/>
 <rectangle x1="45.029746875" y1="35.833471875" x2="45.190846875" y2="35.839440625" layer="21"/>
-<text x="-1.06809375" y="79.713153125" size="1.27" layer="21" font="vector" ratio="12" rot="SR270">XmasCard v1</text>
+<text x="-1.06809375" y="79.713153125" size="1.27" layer="21" font="vector" ratio="12" rot="SR270">XmasCard v1.1</text>
 <text x="39.418003125" y="26.630721875" size="1.27" layer="21" font="vector" ratio="14" rot="SR260" align="center">Colin the Aardvark
 production</text>
 <text x="17.87921875" y="44.673121875" size="1.27" layer="21" font="vector" ratio="14" rot="SR270" align="center">Remove if stored</text>
+<text x="100.78263125" y="46.470996875" size="1.27" layer="21" font="vector" ratio="12" rot="SR270" align="center">CC BY-SA 4.0
+http://github.com/mjholmes</text>
 </plain>
 <attributes>
@@
 </element>
 <element name="S1" library="mjholmes" package="MMS_228_T" value="" x="13.97" y="11.43" rot="R180"/>
+<element name="U$6" library="SparkFun-Aesthetics" package="OSHW-LOGO-M" value="" x="106.1290625" y="47.7181" rot="R270"/>
 </elements>
 <signals>
